File: hardware/HV-schematic.kicad_sch (KiCad schematic)
At the start: 11 parts, among them J10 Power JST, J12 Brake mtr JST, J15 Brake mtr out, J16 Power mtr out, J9 Bat in, U10 ESCON_module-50/5, U11 A4988, U9 Relay

Commit message: Update schematics
Changed lines of the file:
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@@
       (effects (font (size 1.27 1.27)) hide)
     )
-    (property "Value" "" (id 1) (at 69.85 60.96 0))
+    (property "Value" "+24V" (id 1) (at 69.85 60.96 0))
     (property "Footprint" "" (id 2) (at 69.85 64.77 0)
       (effects (font (size 1.27 1.27)) hide)
@@
       (effects (font (size 1.27 1.27)) hide)
     )
-    (property "Value" "" (id 1) (at 83.82 171.45 0))
+    (property "Value" "+24V" (id 1) (at 83.82 171.45 0))
     (property "Footprint" "" (id 2) (at 85.09 175.26 0)
       (effects (font (size 1.27 1.27)) hide)
