File: hardware/LV-schematic.kicad_sch (KiCad schematic)
At the start: 19 parts, among them J1 Brake mtr JST, J2 Aux analog JST, J3 Steer mtr JST, J4 Power JST, J5 On/off JST, J6 Throttle JST, J7 Encoder JST, J8 Steer trq & ang JST, SW1 ON/OFF, U1 Mecostrain2038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

Commit message: Update schematics
Connections:
- net +3V3: no longer U3.16 (3V3), U3.33 (VIN)
- net +5V: now also U3.33 (VIN)
- no-connect marks 92 -> 93
Changed lines of the file:
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@@
   (no_connect (at 77.47 107.95))
   (no_connect (at 77.47 102.87))
+  (no_connect (at 133.35 209.55))
   (no_connect (at 77.47 194.31))
   (no_connect (at 133.35 201.93))
@@
     (stroke (width 0) (type default) (color 0 0 0 0))
   )
-  (wire (pts (xy 133.35 209.55) (xy 138.43 209.55))
-    (stroke (width 0) (type default) (color 0 0 0 0))
-  )
   (wire (pts (xy 44.45 29.21) (xy 68.58 29.21))
     (stroke (width 0) (type default) (color 0 0 0 0))
@@
   )
   (wire (pts (xy 77.47 88.9) (xy 67.31 88.9))
-    (stroke (width 0) (type default) (color 0 0 0 0))
-  )
-  (wire (pts (xy 138.43 205.74) (xy 138.43 209.55))
     (stroke (width 0) (type default) (color 0 0 0 0))
   )
@@
     (pin "5")
     (pin "6")
-  )
-  (symbol (lib_id "power:+3V3") (at 72.39 226.06 0) (unit 1)
-    (in_bom yes) (on_board yes)
-    (property "Reference" "#PWR0102" (id 0) (at 72.39 229.87 0)
-      (effects (font (size 1.27 1.27)) hide)
-    )
-    (property "Value" "+3V3" (id 1) (at 72.39 222.25 0))
-    (property "Footprint" "" (id 2) (at 72.39 226.06 0)
-      (effects (font (size 1.27 1.27)) hide)
-    )
-    (property "Datasheet" "" (id 3) (at 72.39 226.06 0)
-      (effects (font (size 1.27 1.27)) hide)
-    )
-    (pin "1")
   )
   (symbol (lib_id "power:GND") (at 46.99 50.8 90) (mirror x) (unit 1)
@@
     (pin "5")
   )
-  (symbol (lib_id "power:+3V3") (at 138.43 205.74 0) (mirror y) (unit 1)
-    (in_bom yes) (on_board yes)
-    (property "Reference" "#PWR0103" (id 0) (at 138.43 209.55 0)
-      (effects (font (size 1.27 1.27)) hide)
-    )
-    (property "Value" "+3V3" (id 1) (at 138.43 201.93 0))
-    (property "Footprint" "" (id 2) (at 138.43 205.74 0)
-      (effects (font (size 1.27 1.27)) hide)
-    )
-    (property "Datasheet" "" (id 3) (at 138.43 205.74 0)
-      (effects (font (size 1.27 1.27)) hide)
-    )
-    (pin "1")
-  )
   (symbol (lib_id "power:GND") (at 77.47 33.02 270) (mirror x) (unit 1)
     (in_bom yes) (on_board yes) (fields_autoplaced)
@@
       (effects (font (size 1.27 1.27)) hide)
     )
+    (pin "1")
+  )
+  (symbol (lib_id "power:+5V") (at 72.39 226.06 0) (mirror y) (unit 1)
+    (in_bom yes) (on_board yes)
+    (property "Reference" "#PWR?" (id 0) (at 72.39 229.87 0)
+      (effects (font (size 1.27 1.27)) hide)
+    )
+    (property "Value" "+5V" (id 1) (at 74.93 222.25 0)
+      (effects (font (size 1.27 1.27)) (justify left))
+    )
+    (property "Footprint" "" (id 2) (at 72.39 226.06 0)
+      (effects (font (size 1.27 1.27)) hide)
+    )
+    (property "Datasheet" "" (id 3) (at 72.39 226.06 0)
+      (effects (font (size 1.27 1.27)) hide)
+    )

Commit message: Update schematics
Connections:
- net +3V3: no longer U7.2 (VCC), U8.2 (VCC)
- net +5V: now also U7.2 (VCC)
- net at U7.9 (3V3): now also U8.2 (VCC)
- no-connect marks 93 -> 92
Changed lines of the file:
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@@
     (comment 1 "Low-voltage motherboard schematic")
   )
-  (junction (at 156.21 104.14) (diameter 0) (color 0 0 0 0)
-  )
   (junction (at 107.95 146.05) (diameter 0) (color 0 0 0 0)
   )
@@
   )
   (junction (at 57.15 177.8) (diameter 0) (color 0 0 0 0)
-  )
-  (junction (at 156.21 80.01) (diameter 0) (color 0 0 0 0)
   )
   (junction (at 156.21 55.88) (diameter 0) (color 0 0 0 0)
@@
   (no_connect (at 77.47 191.77))
   (no_connect (at 77.47 204.47))
+  (no_connect (at 177.8 107.95))
   (no_connect (at 177.8 29.21))
   (no_connect (at 133.35 43.18))
@@
   (no_connect (at 133.35 219.71))
   (no_connect (at 85.09 146.05))
-  (no_connect (at 177.8 107.95))
   (no_connect (at 77.47 100.33))
   (no_connect (at 77.47 176.53))
@@
   (no_connect (at 160.02 134.62))
   (no_connect (at 133.35 71.12))
-  (no_connect (at 177.8 110.49))
   (no_connect (at 133.35 105.41))
   (no_connect (at 77.47 186.69))
@@
     (stroke (width 0) (type default) (color 0 0 0 0))
   )
+  (wire (pts (xy 156.21 119.38) (xy 156.21 132.08))
+    (stroke (width 0) (type default) (color 0 0 0 0))
+  )
   (wire (pts (xy 156.21 55.88) (xy 156.21 80.01))
     (stroke (width 0) (type default) (color 0 0 0 0))
@@
     (stroke (width 0) (type default) (color 0 0 0 0))
   )
+  (wire (pts (xy 177.8 110.49) (xy 180.34 110.49))
+    (stroke (width 0) (type default) (color 0 0 0 0))
+  )
   (wire (pts (xy 107.95 146.05) (xy 113.03 146.05))
     (stroke (width 0) (type default) (color 0 0 0 0))
@@
     (stroke (width 0) (type default) (color 0 0 0 0))
   )
-  (wire (pts (xy 160.02 132.08) (xy 156.21 132.08))
-    (stroke (width 0) (type default) (color 0 0 0 0))
-  )
   (wire (pts (xy 148.59 27.94) (xy 148.59 24.13))
     (stroke (width 0) (type default) (color 0 0 0 0))
@@
     (stroke (width 0) (type default) (color 0 0 0 0))
   )
-  (wire (pts (xy 156.21 80.01) (xy 156.21 104.14))
-    (stroke (width 0) (type default) (color 0 0 0 0))
-  )
   (wire (pts (xy 152.4 85.09) (xy 160.02 85.09))
     (stroke (width 0) (type default) (color 0 0 0 0))
@@
     (stroke (width 0) (type default) (color 0 0 0 0))
   )
-  (wire (pts (xy 156.21 132.08) (xy 156.21 104.14))
-    (stroke (width 0) (type default) (color 0 0 0 0))
-  )
   (wire (pts (xy 64.77 76.2) (xy 64.77 58.42))
     (stroke (width 0) (type default) (color 0 0 0 0))
@@
     (stroke (width 0) (type default) (color 0 0 0 0))
   )
-  (wire (pts (xy 160.02 104.14) (xy 156.21 104.14))
-    (stroke (width 0) (type default) (color 0 0 0 0))
-  )
   (wire (pts (xy 57.15 177.8) (xy 57.15 181.61))
     (stroke (width 0) (type default) (color 0 0 0 0))
@@
     (stroke (width 0) (type default) (color 0 0 0 0))
   )
-  (wire (pts (xy 181.61 105.41) (xy 181.61 121.92))
+  (wire (pts (xy 182.88 105.41) (xy 182.88 121.92))
+    (stroke (width 0) (type default) (color 0 0 0 0))
+  )
+  (wire (pts (xy 180.34 119.38) (xy 156.21 119.38))
     (stroke (width 0) (type default) (color 0 0 0 0))
   )
@@
     (stroke (width 0) (type default) (color 0 0 0 0))
   )
-  (wire (pts (xy 181.61 121.92) (xy 113.03 121.92))
+  (wire (pts (xy 182.88 121.92) (xy 113.03 121.92))
     (stroke (width 0) (type default) (color 0 0 0 0))
   )
@@
     (stroke (width 0) (type default) (color 0 0 0 0))
   )
-  (wire (pts (xy 177.8 105.41) (xy 181.61 105.41))
+  (wire (pts (xy 177.8 105.41) (xy 182.88 105.41))
     (stroke (width 0) (type default) (color 0 0 0 0))
   )
@@
     (stroke (width 0) (type default) (color 0 0 0 0))
   )
+  (wire (pts (xy 156.21 132.08) (xy 160.02 132.08))
+    (stroke (width 0) (type default) (color 0 0 0 0))
+  )
   (wire (pts (xy 44.45 83.82) (xy 50.8 83.82))
     (stroke (width 0) (type default) (color 0 0 0 0))
@@
     (stroke (width 0) (type default) (color 0 0 0 0))
   )
+  (wire (pts (xy 180.34 110.49) (xy 180.34 119.38))
+    (stroke (width 0) (type default) (color 0 0 0 0))
+  )
   (wire (pts (xy 57.15 177.8) (xy 44.45 177.8))
     (stroke (width 0) (type default) (color 0 0 0 0))
@@
     (stroke (width 0) (type default) (color 0 0 0 0))
   )
+  (wire (pts (xy 154.94 104.14) (xy 154.94 100.33))
+    (stroke (width 0) (type default) (color 0 0 0 0))
+  )
   (wire (pts (xy 67.31 60.96) (xy 67.31 78.74))
     (stroke (width 0) (type default) (color 0 0 0 0))
@@
   )
   (wire (pts (xy 77.47 30.48) (xy 73.66 30.48))
+    (stroke (width 0) (type default) (color 0 0 0 0))
+  )
+  (wire (pts (xy 160.02 104.14) (xy 154.94 104.14))
     (stroke (width 0) (type default) (color 0 0 0 0))
   )
@@
     (pin "4")
   )
+  (symbol (lib_id "power:+5V") (at 154.94 100.33 0) (mirror y) (unit 1)
+    (in_bom yes) (on_board yes)
+    (property "Reference" "#PWR?" (id 0) (at 154.94 104.14 0)
+      (effects (font (size 1.27 1.27)) hide)
+    )
+    (property "Value" "+5V" (id 1) (at 157.48 96.52 0)
+      (effects (font (size 1.27 1.27)) (justify left))
+    )
+    (property "Footprint" "" (id 2) (at 154.94 100.33 0)
+      (effects (font (size 1.27 1.27)) hide)
+    )
+    (property "Datasheet" "" (id 3) (at 154.94 100.33 0)
+      (effects (font (size 1.27 1.27)) hide)
+    )
+    (pin "1")
+  )
   (symbol (lib_id "power:GND") (at 81.28 137.16 0) (mirror x) (unit 1)
